Commit message: feat(gazebo): 仿真巡线，line_track 支持从图像话题取图
- line_track 新增 image_topic 参数:为空仍走 USB 摄像头(行为不变),
  设置后改订阅该 sensor_msgs/Image 话题(cv_bridge),真车/仿真通用
- 新增巡线世界 yahboom_line.world(地面黄色曲线)、line_follow_sim.launch.py、
  黄线 HSV 阈值 config/line_hsv_sim.txt
- gazebo xacro 增加 camera_pitch 参数,巡线时相机俯视
- 容器内用 xvfb + 软件GL headless 实测跑通:相机出图、每帧识别到线、
  机器人沿曲线行驶,跟踪误差约几厘米

https://claude.ai/code/session_018dVoVDwzWxEiXuzBpVhZWY

File: src/yahboomcar_gazebo/urdf/yahboomcar_X3_gazebo.urdf.xacro (robot description, xacro)
@@ -10,4 +10,8 @@
 -->
 <robot name="yahboomcar" xmlns:xacro="http://wiki.ros.org/xacro">
+    <!-- Pitch (rad) applied to the camera sensor only (not the TF frame); a
+         positive value tilts the optical axis downward for line following. -->
+    <xacro:arg name="camera_pitch" default="0.0"/>
+    <xacro:property name="camera_pitch" value="$(arg camera_pitch)"/>
     <xacro:property name="mesh_pkg" value="package://yahboomcar_description/meshes"/>
     <material name="Green"><color rgba="0 0.7 0 1"/></material>
@@ -241,4 +245,5 @@
     <gazebo reference="camera_link">
         <sensor name="camera_sensor" type="camera">
+            <pose>0 0 0 0 ${camera_pitch} 0</pose>
             <always_on>true</always_on>
             <update_rate>30</update_rate>
